Commit message: added world of simple sidewalk intersection

File: hambot_sim_ws/src/hambot_description/urdf/hambot.urdf.xacro (robot description, xacro)
@@ -118,5 +118,5 @@
     <parent link="base_link"/>
     <child link="oak_d_lite_frame"/>
-    <origin xyz="0.23 0 0.03" rpy="0 0 0"/>
+    <origin xyz="0.23 0 0.09" rpy="0 0 0"/>
   </joint>
   <gazebo reference="oak_d_lite_frame">

Commit message: Changed the descriptor to look more similar to the hambot we have

File: hambot_sim_ws/src/hambot_description/urdf/hambot.urdf.xacro (robot description, xacro)
@@ -1,4 +1,32 @@
 <?xml version="1.0"?>
 <robot xmlns:xacro="http://www.ros.org/wiki/xacro" name="hambot">
+  <!-- ========================================== -->
+  <!-- 0. CONFIGURABLE SPECIFIC PROPERTIES        -->
+  <!-- ========================================== -->
+  <!-- Chassis Dimensions -->
+  <xacro:property name="chassis_len"   value="0.193"/>  <!-- 193 mm -->
+  <xacro:property name="chassis_width" value="0.157"/>  <!-- 157 mm -->
+  <xacro:property name="chassis_hgt"   value="0.100"/>  <!-- 100 mm -->
+  <xacro:property name="chassis_mass"  value="2.5"/>
+  <!-- Wheel Dimensions & Placement -->
+  <xacro:property name="wheel_rad"     value="0.045"/>  <!-- 45 mm radius -->
+  <xacro:property name="wheel_len"     value="0.010"/>  <!-- 10 mm thickness -->
+  <xacro:property name="wheel_mass"    value="0.15"/>
+  <xacro:property name="wheel_joint_y" value="0.0995"/> <!-- 16mm clearance from chassis side -->
+  <xacro:property name="wheel_joint_x" value="0.051"/>  <!-- 12mm clearance between wheels -->
+  <!-- Ground Clearance & Coordinate Math -->
+  <xacro:property name="base_link_z_offset" value="0.071"/> <!-- Ground clearance 21mm + half chassis height -->
+  <xacro:property name="wheel_joint_z"      value="${wheel_rad - base_link_z_offset}"/> <!-- -26 mm relative to base_link -->
+  <!-- Camera Stand (Support) -->
+  <xacro:property name="stand_len"     value="0.010"/>  <!-- 10 mm -->
+  <xacro:property name="stand_width"   value="0.092"/>  <!-- 92 mm -->
+  <xacro:property name="stand_hgt"     value="0.250"/>  <!-- 250 mm -->
+  <xacro:property name="stand_joint_x" value="-0.0915"/> <!-- Positioned at the rear end of chassis -->
+  <!-- Camera -->
+  <xacro:property name="camera_len"     value="0.015"/> <!-- 15 mm -->
+  <xacro:property name="camera_width"   value="0.090"/> <!-- 90 mm -->
+  <xacro:property name="camera_hgt"     value="0.025"/> <!-- 25 mm -->
+  <xacro:property name="camera_joint_z" value="0.220"/> <!-- 220 mm above top of chassis -->
+  <xacro:property name="camera_joint_x" value="0.0125"/> <!-- Flush on front face of the stand -->
   <!-- ========================================== -->
   <!-- 1. MATERIALS & INERTIAL MACROS             -->
@@ -30,15 +58,15 @@
     <parent link="base_footprint"/>
     <child link="base_link"/>
-    <origin xyz="0 0 0.1" rpy="0 0 0"/>
+    <origin xyz="0 0 ${base_link_z_offset}" rpy="0 0 0"/>
   </joint>
   <link name="base_link">
     <visual>
-      <geometry><box size="0.5 0.3 0.15"/></geometry>
+      <geometry><box size="${chassis_len} ${chassis_width} ${chassis_hgt}"/></geometry>
       <material name="blue"/>
     </visual>
     <collision>
-      <geometry><box size="0.5 0.3 0.15"/></geometry>
-    </collision>
-    <xacro:box_inertia m="5.0" w="0.5" h="0.3" d="0.15"/>
+      <geometry><box size="${chassis_len} ${chassis_width} ${chassis_hgt}"/></geometry>
+    </collision>
+    <xacro:box_inertia m="${chassis_mass}" w="${chassis_len}" h="${chassis_width}" d="${chassis_hgt}"/>
   </link>
   <!-- ========================================== -->
@@ -49,16 +77,16 @@
       <parent link="base_link"/>
       <child link="${prefix}_wheel"/>
-      <origin xyz="${x_reflect*0.18} ${y_reflect*0.18} -0.05" rpy="${-pi/2} 0 0"/>
+      <origin xyz="${x_reflect*wheel_joint_x} ${y_reflect*wheel_joint_y} ${wheel_joint_z}" rpy="${-pi/2} 0 0"/>
       <axis xyz="0 0 1"/>
     </joint>
     <link name="${prefix}_wheel">
       <visual>
-        <geometry><cylinder radius="0.1" length="0.05"/></geometry>
+        <geometry><cylinder radius="${wheel_rad}" length="${wheel_len}"/></geometry>
         <material name="black"/>
       </visual>
       <collision>
-        <geometry><cylinder radius="0.1" length="0.05"/></geometry>
+        <geometry><cylinder radius="${wheel_rad}" length="${wheel_len}"/></geometry>
       </collision>
-      <xacro:cylinder_inertia m="0.5" r="0.1" h="0.05"/>
+      <xacro:cylinder_inertia m="${wheel_mass}" r="${wheel_rad}" h="${wheel_len}"/>
     </link>
   </xacro:macro>
@@ -70,16 +98,22 @@
   <!-- 4. SIMULATED SENSORS                       -->
   <!-- ========================================== -->
-  <!-- LiDAR Frame & Gazebo Sensor -->
+  <!-- LiDAR Frame & Gazebo Sensor (Located in the Center on Top of Chassis) -->
   <link name="laser_frame">
     <visual>
-      <geometry><cylinder radius="0.05" length="0.05"/></geometry>
+      <!-- Shifted visual cylinder origin up by half its height so it sits on top of chassis -->
+      <origin xyz="0 0 0.02" rpy="0 0 0"/>
+      <geometry><cylinder radius="0.03" length="0.04"/></geometry>
       <material name="grey"/>
     </visual>
-    <xacro:cylinder_inertia m="0.1" r="0.05" h="0.05"/>
+    <collision>
+      <origin xyz="0 0 0.02" rpy="0 0 0"/>
+      <geometry><cylinder radius="0.03" length="0.04"/></geometry>
+    </collision>
+    <xacro:cylinder_inertia m="0.1" r="0.03" h="0.04"/>
   </link>
   <joint name="laser_joint" type="fixed">
     <parent link="base_link"/>
     <child link="laser_frame"/>
-    <origin xyz="0.15 0 0.1" rpy="0 0 0"/>
+    <origin xyz="0 0 ${chassis_hgt/2}" rpy="0 0 0"/>
   </joint>
   <gazebo reference="laser_frame">
@@ -107,22 +141,58 @@
     </sensor>
   </gazebo>
-  <!-- OAK-D Lite Depth Camera Frame & Gazebo Sensor -->
-  <link name="oak_d_lite_frame">
-    <visual>
-      <geometry><box size="0.02 0.1 0.03"/></geometry>
+  <!-- Camera Stand (Support Mast) -->
+  <link name="camera_stand">
+    <visual>
+      <!-- Visual geometry origin shifted up so the bottom of the stand aligns with the joint link origin -->
+      <origin xyz="0 0 ${stand_hgt/2}" rpy="0 0 0"/>
+      <geometry>
+        <box size="${stand_len} ${stand_width} ${stand_hgt}"/>
+      </geometry>
+      <material name="grey"/>
+    </visual>
+    <collision>
+      <origin xyz="0 0 ${stand_hgt/2}" rpy="0 0 0"/>
+      <geometry>
+        <box size="${stand_len} ${stand_width} ${stand_hgt}"/>
+      </geometry>
+    </collision>
+    <xacro:box_inertia m="0.15" w="${stand_len}" h="${stand_width}" d="${stand_hgt}"/>
+  </link>
+  <joint name="stand_joint" type="fixed">
+    <parent link="base_link"/>
+    <child link="camera_stand"/>
+    <origin xyz="${stand_joint_x} 0 ${chassis_hgt/2}" rpy="0 0 0"/>
+  </joint>
+  <!-- Camera Frame & Gazebo Sensor -->
+  <link name="camera_frame">
+    <visual>
+      <geometry>
+        <box size="${camera_len} ${camera_width} ${camera_hgt}"/>
+      </geometry>
       <material name="black"/>
     </visual>
-    <xacro:box_inertia m="0.05" w="0.02" h="0.1" d="0.03"/>
+    <collision>
+      <geometry>
+        <box size="${camera_len} ${camera_width} ${camera_hgt}"/>
+      </geometry>
+    </collision>
+    <xacro:box_inertia m="0.05" w="${camera_len}" h="${camera_width}" d="${camera_hgt}"/>
   </link>
   <joint name="camera_joint" type="fixed">
+<<<<<<< HEAD
     <parent link="base_link"/>
     <child link="oak_d_lite_frame"/>
     <origin xyz="0.23 0 0.09" rpy="0 0 0"/>
-  </joint>
-  <gazebo reference="oak_d_lite_frame">
+=======
+    <parent link="camera_stand"/>
+    <child link="camera_frame"/>
+    <origin xyz="${camera_joint_x} 0 ${camera_joint_z}" rpy="0 0 0"/>
+>>>>>>> 2aa524b (Changed the descriptor to look more similar to the)
+  </joint>
+  <gazebo reference="camera_frame">
     <sensor name="camera" type="rgbd_camera">
       <pose>0 0 0 0 0 0</pose>
       <topic>camera</topic>
-      <update_rate>5</update_rate> <!-- lowerd this to 5 for performance can change to 30 for real comparisons -->
+      <update_rate>5</update_rate>
       <camera>
         <horizontal_fov>1.274</horizontal_fov>
@@ -149,6 +219,7 @@
       <right_joint>front_right_wheel_joint</right_joint>
       <right_joint>rear_right_wheel_joint</right_joint>
-      <wheel_separation>0.36</wheel_separation>
-      <wheel_radius>0.1</wheel_radius>
+      <!-- Automatically calculated from variables to maintain accurate physical values -->
+      <wheel_separation>${wheel_joint_y * 2}</wheel_separation>
+      <wheel_radius>${wheel_rad}</wheel_radius>
       <odom_publish_frequency>30</odom_publish_frequency>
       <topic>cmd_vel</topic>
@@ -158,5 +229,4 @@
       <child_frame_id>base_footprint</child_frame_id>
     </plugin>
-    <!-- Essential plugin to publish all moving joint positions to ROS 2 -->
     <plugin filename="ignition-gazebo-joint-state-publisher-system" name="ignition::gazebo::systems::JointStatePublisher">
       <topic>joint_states</topic>

Commit message: Accepted incoming changes

File: hambot_sim_ws/src/hambot_description/urdf/hambot.urdf.xacro (robot description, xacro)
@@ -180,13 +180,7 @@
   </link>
   <joint name="camera_joint" type="fixed">
-<<<<<<< HEAD
-    <parent link="base_link"/>
-    <child link="oak_d_lite_frame"/>
-    <origin xyz="0.23 0 0.09" rpy="0 0 0"/>
-=======
     <parent link="camera_stand"/>
     <child link="camera_frame"/>
     <origin xyz="${camera_joint_x} 0 ${camera_joint_z}" rpy="0 0 0"/>
->>>>>>> 2aa524b (Changed the descriptor to look more similar to the)
   </joint>
   <gazebo reference="camera_frame">

Commit message: added simulated imu module added ros robot localization node package to docker

File: hambot_sim_ws/src/hambot_description/urdf/hambot.urdf.xacro (robot description, xacro)
@@ -164,4 +164,24 @@
     <origin xyz="${stand_joint_x} 0 ${chassis_hgt/2}" rpy="0 0 0"/>
   </joint>
+  <!-- IMU Frame (center of chassis) -->
+  <link name="imu_frame">
+    <inertial>
+      <mass value="0.01"/>
+      <inertia ixx="1e-6" ixy="0.0" ixz="0.0" iyy="1e-6" iyz="0.0" izz="1e-6"/>
+    </inertial>
+  </link>
+  <joint name="imu_joint" type="fixed">
+    <parent link="base_link"/>
+    <child link="imu_frame"/>
+    <origin xyz="0 0 ${chassis_hgt/2}" rpy="0 0 0"/>
+  </joint>
+  <gazebo reference="imu_frame">
+    <sensor name="imu_sensor" type="imu">
+      <topic>/imu/data</topic>
+      <update_rate>50</update_rate>
+      <always_on>1</always_on>
+      <visualize>true</visualize>
+    </sensor>
+  </gazebo>
   <!-- Camera Frame & Gazebo Sensor -->
   <link name="camera_frame">
